Commit message: add action reward. move aubo to (-0.5 0 0), and add debug comment

File: aubo_robot/aubo_gazebo/urdf/aubo_i5.urdf (robot description, URDF)
Before this commit: robot aubo_i5, 21 links, 20 joints
Joints:
- joint world_joint: origin xyz=0.0 0.0 0.1 rpy=0.0 0.0 0.0 -> xyz=-0.5 0.0 0.1 rpy=0.0 0.0 0.0

File: aubo_robot/aubo_gazebo/urdf/aubo_i5_with_gripper.urdf (robot description, URDF)
Before this commit: robot aubo_i5, 21 links, 20 joints
Joints:
- joint world_joint: origin xyz=-0.5 0.0 0.1 rpy=0.0 0.0 0.0 -> xyz=0. 0.0 0.1 rpy=0.0 0.0 0.0
