Commit message: add sample_gaol function and goal orientatoin. observation is dict spaces like fetch

File: aubo_robot/aubo_gazebo/urdf/aubo_i5_with_gripper.urdf (robot description, URDF)
Before this commit: robot aubo_i5, 21 links, 20 joints
Joints:
- joint world_joint: origin xyz=0.0 0.0 0.1 rpy=0.0 0.0 0.0 -> xyz=-0.5 0.0 0.1 rpy=0.0 0.0 0.0

Commit message: add action_reward reduction index, uncomment debug log

File: aubo_robot/aubo_gazebo/urdf/aubo_i5_with_gripper.urdf (robot description, URDF)
Before this commit: robot aubo_i5, 21 links, 20 joints
Joints:
- joint world_joint: origin xyz=0. 0.0 0.1 rpy=0.0 0.0 0.0 -> xyz=-0.5 0.0 0.1 rpy=0.0 0.0 0.0
